File: hardware/attiny84_tester-mk-1.0.brd (EAGLE design)
At the start: 32 x 44 mm, 27 parts, among them IC1 ATTiny84

Commit message: and now add in revision info since i'm bound to want that later
Other:
- board text added: ">VERSION"
- board text added: "Rev"
Changed lines of the file:
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@@
 <text x="16" y="2.75" size="0.6" layer="22" font="vector" ratio="16" rot="MR0" align="top-center">by schizobovine
 &lt;sean@yak.net&gt;</text>
+<text x="6.25" y="2" size="1" layer="21" font="vector" ratio="16" align="center">&gt;VERSION</text>
+<text x="6.25" y="2" size="1" layer="1" font="vector" ratio="16" align="center">&gt;VERSION</text>
+<text x="6.25" y="3.25" size="1" layer="21" font="vector" ratio="16" align="center">Rev</text>
+<text x="6.25" y="3.25" size="1" layer="1" font="vector" ratio="16" align="center">Rev</text>
+<text x="26" y="41" size="1" layer="22" font="vector" ratio="16" rot="MR0" align="center">&gt;VERSION</text>
+<text x="26" y="41" size="1" layer="16" font="vector" ratio="16" rot="MR0" align="center">&gt;VERSION</text>
+<text x="26" y="42.25" size="1" layer="22" font="vector" ratio="16" rot="MR0" align="center">Rev</text>
+<text x="26" y="42.25" size="1" layer="16" font="vector" ratio="16" rot="MR0" align="center">Rev</text>
 </plain>
 <attributes>
+<attribute name="VERSION" value="1.0"/>
 </attributes>
 <variantdefs>
@@
 <elements>
 <element name="FRAME1" library="A_butts" package="DUMMY" value="" x="0.5" y="0.5" smashed="yes">
-<attribute name="VERSION" value="v01" x="0.5" y="0.5" size="0.5" layer="27" ratio="12" display="off"/>
-<attribute name="DESIGNER" value="Nobody" x="0.5" y="0.5" size="0.5" layer="27" ratio="12" display="off"/>
+<attribute name="VERSION" value="1.0" x="0.5" y="0.5" size="0.5" layer="27" ratio="12" display="off"/>
+<attribute name="DESIGNER" value="sean@yak.net" x="0.5" y="0.5" size="0.5" layer="27" ratio="12" display="off"/>
 </element>
 <element name="IC1" library="A_butts" package="ZIF14" value="ATTiny84" x="16" y="25.5" smashed="yes" rot="R270">
@@
 <attribute name="MF" value="3M" x="16" y="25.5" size="0.5" layer="27" ratio="12" rot="R270" display="off"/>
 <attribute name="OC_FARNELL" value="1247151" x="16" y="25.5" size="0.5" layer="27" ratio="12" rot="R270" display="off"/>
-<attribute name="NAME" x="24.034" y="42.5" size="0.8" layer="25" font="vector" ratio="12" rot="R270" align="bottom-center"/>
+<attribute name="NAME" x="7.284" y="13.75" size="0.8" layer="25" font="vector" ratio="12" rot="SR270" align="bottom-center"/>
 <attribute name="VALUE" x="16" y="25.5" size="1" layer="21" font="vector" ratio="16" rot="SR270" align="center"/>
 </element>

Commit message: changed names to be more helpful
Parts:
- renumbered LED10 to D8, LED11 to D9, LED12 to D10, LED2 to D0, LED3 to D1, LED4 to D2, LED5 to D3, LED6 to D4, LED7 to D5, LED8 to D6, LED9 to D7
